File: reflectancesensor/reflectancesensors.kicad_pcb (KiCad board)
At the start: 2 copper layers, 62 x 47 mm, 18 parts, among them J2 Conn_01x04_Socket, Q1 BPW40, Q2 BPW40, U1 TCRT5000L, U3 TCRT5000L

Commit message: Some fixes
Parts:
- removed REF**: , GS_Virtual:ENPH253_Logo_Small
- added S1: Logo, GS_Virtual:ENPH253_Logo, F.Cu at (102.2, 124.0)
- J2: footprint Connector_JST:JST_XH_S4B-XH-A-1_1x04_P2.50mm_Horizontal -> GS_Connectors:JST_XH_S4B-XH-A-1_1x04_P2.50mm_Horizontal
Connections:
- J2 pad 1: +3V3 -> GND
- J2 pad 4: GND -> +3V3
- Q1 pad 1: Net-(J2-Pin_2) -> Net-(J2-Pin_3)
- Q2 pad 1: Net-(J2-Pin_3) -> Net-(J2-Pin_2)
- RV1 pad 2: Net-(J2-Pin_2) -> Net-(J2-Pin_3)
- RV2 pad 2: Net-(J2-Pin_3) -> Net-(J2-Pin_2)
- U1 pad 1: Net-(J2-Pin_2) -> Net-(J2-Pin_3)
- U3 pad 1: Net-(J2-Pin_3) -> Net-(J2-Pin_2)
Routing:
- net +3V3: track 34.9 -> 67.0 mm
- net Net-(J2-Pin_2): track 67.5 -> 54.8 mm
- net GND: vias 79 -> 74
Other:
- board text added: "3V3"
- board text added: "GND"
- board text added: "IR0"
- board text added: "IR1"
