File: reflectancesensor/reflectancesensors.kicad_sch (KiCad schematic)
At the start: 17 parts, among them J2 Conn_01x04_Socket, Q1 BPW40, Q2 BPW40, U1 TCRT5000L, U3 TCRT5000L

Commit message: Some fixes
Parts:
- added S1: Logo, GS_Virtual:ENPH253_Logo, symbol GS_Virtual:ENPH253_Logo
- J2: footprint Connector_JST:JST_XH_S4B-XH-A-1_1x04_P2.50mm_Horizontal -> GS_Connectors:JST_XH_S4B-XH-A-1_1x04_P2.50mm_Horizontal
Connections:
- net +3V3: now also J2.4 (Pin_4); no longer J2.1 (Pin_1)
- net GND: now also J2.1 (Pin_1); no longer J2.4 (Pin_4)
- net at Q1.1 (C), RV1.2, U1.1: now also J2.3 (Pin_3); no longer J2.2 (Pin_2)
- net at Q2.1 (C), RV2.2, U3.1: now also J2.2 (Pin_2); no longer J2.3 (Pin_3)
Changed lines of the file:
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@@
+	(wire
+		(pts
+			(xy 184.15 31.75) (xy 184.15 90.17)
+		)
+		(stroke
+			(width 0)
+			(type default)
+		)
+	)
 	(wire
 		(pts
@@
 	(wire
 		(pts
-			(xy 184.15 31.75) (xy 184.15 90.17)
-		)
-		(stroke
-			(width 0)
-			(type default)
-		)
-	)
-	(wire
-		(pts
 			(xy 67.31 156.21) (xy 68.58 156.21)
 		)
@@
 	(wire
 		(pts
-			(xy 184.15 156.21) (xy 184.15 97.79)
+			(xy 184.15 97.79) (xy 184.15 156.21)
 		)
 		(stroke
@@
 	)
 	(symbol
+		(lib_id "GS_Virtual:ENPH253_Logo")
+		(at 170.18 194.31 0)
+		(unit 1)
+		(exclude_from_sim no)
+		(in_bom no)
+		(on_board yes)
+		(dnp no)
+		(fields_autoplaced yes)
+		(property "Reference" "S1"
+			(at 170.18 190.5 0)
+			(effects
+				(font
+					(size 1.27 1.27)
+				)
+			)
+		)
+		(property "Value" "Logo"
+			(at 170.18 185.928 0)
+			(effects
+				(font
+					(size 1.27 1.27)
+				)
+				(hide yes)
+			)
+		)
+		(property "Footprint" "GS_Virtual:ENPH253_Logo"
+			(at 170.18 194.31 0)
+			(effects
+				(font
+					(size 1.27 1.27)
+				)
+				(hide yes)
+			)
+		)
+		(property "Datasheet" ""
+			(at 170.18 194.31 0)
+			(effects
+				(font
+					(size 1.27 1.27)
+				)
+				(hide yes)
+			)
+		)
+		(property "Description" "ENPH 253 Team Logo"
+			(at 170.18 188.214 0)
+			(effects
+				(font
+					(size 1.27 1.27)
+				)
+				(hide yes)
+			)
+		)
+		(instances
+			(project ""
+				(path "/6ca5ba81-b900-4043-9a89-71bd4e9b2915"
+					(reference "S1")
+					(unit 1)
+				)
+			)
+		)
+	)
+	(symbol
 		(lib_id "Device:C_Polarized")
 		(at 71.12 40.64 0)
@@
 	(symbol
 		(lib_id "Connector:Conn_01x04_Socket")
-		(at 189.23 92.71 0)
+		(at 189.23 95.25 0)
+		(mirror x)
 		(unit 1)
 		(exclude_from_sim no)
@@
 		(on_board yes)
 		(dnp no)
-		(fields_autoplaced yes)
 		(property "Reference" "J2"
-			(at 190.5 92.7099 0)
+			(at 190.5 95.2501 0)
 			(effects
 				(font
@@
 		)
 		(property "Value" "Conn_01x04_Socket"
-			(at 190.5 95.2499 0)
+			(at 190.5 92.7101 0)
 			(effects
 				(font
@@
 			)
 		)
-		(property "Footprint" "Connector_JST:JST_XH_S4B-XH-A-1_1x04_P2.50mm_Horizontal"
-			(at 189.23 92.71 0)
+		(property "Footprint" "GS_Connectors:JST_XH_S4B-XH-A-1_1x04_P2.50mm_Horizontal"
+			(at 189.23 95.25 0)
 			(effects
 				(font
@@
 		)
 		(property "Datasheet" "~"
-			(at 189.23 92.71 0)
+			(at 189.23 95.25 0)
 			(effects
 				(font
@@
 		)
 		(property "Description" "Generic connector, single row, 01x04, script generated"
-			(at 189.23 92.71 0)
-			(effects
-				(font
+			(at 189.23 95.25 0)
+			(effects
+				(font
